Commit message: wip: trying to get points published (working) to show up visually in rviz which isnt working

File: src/drone_viz/urdf/drone_arena.urdf (robot description, URDF)
Before this commit: robot drone_arena, 2 links, 1 joints
Links:
- link arena: geometry visual box size=6.7056 5.4864 2.7432
Joints:
- joint base_to_arena: origin xyz=0 0 -1.524 rpy=0 0 0 -> xyz=0 0 -1.3716 rpy=0 0 0
