Commit message: prog: drone showing, need to update the pose of it

File: src/drone_viz/urdf/drone_arena.xacro (robot description, xacro)
@@ -23,5 +23,5 @@
       <visual>
         <geometry>
-          <mesh filename="package://drone_viz/meshes/crazyflie.stl" scale="0.001 0.001 0.001"/>
+          <mesh filename="package://drone_viz/meshes/crazyflie.stl" scale="0.01 0.01 0.01"/>
         </geometry>
         <material name="gray">

Commit message: feat: drone showing and updating pose rt!

File: src/drone_viz/urdf/drone_arena.xacro (robot description, xacro)
@@ -1,7 +1,7 @@
 <?xml version="1.0"?>
 <robot xmlns:xacro="http://ros.org/wiki/xacro" name="drone_arena">
-  <!-- Arena volume box (visual only) -->
   <link name="arena">
     <visual>
+      <origin xyz="0 0 0" rpy="0 0 0"/>
       <geometry>
         <box size="6.7056 5.4864 2.7432"/>
@@ -12,29 +12,15 @@
     </visual>
   </link>
-  <link name="base_link"/>
+  <link name="base_link">
+    <visual>
+      <geometry>
+        <mesh filename="package://drone_viz/meshes/crazyflie.stl" scale="0.01 0.01 0.01"/>
+      </geometry>
+    </visual>
+  </link>
   <joint name="base_to_arena" type="fixed">
     <parent link="arena"/>
     <child link="base_link"/>
-    <origin xyz="0 0 -1.3716" rpy="0 0 0"/>
+    <origin xyz="0 0 -2.7432" rpy="0 0 0"/>
   </joint>
-  <!-- Drone macro -->
-  <xacro:macro name="drone" params="id">
-    <link name="drone_${id}">
-      <visual>
-        <geometry>
-          <mesh filename="package://drone_viz/meshes/crazyflie.stl" scale="0.01 0.01 0.01"/>
-        </geometry>
-        <material name="gray">
-          <color rgba="0.5 0.5 0.5 1"/>
-        </material>
-      </visual>
-    </link>
-    <joint name="drone_${id}_tf_joint" type="floating">
-      <parent link="base_link"/>
-      <child link="drone_${id}"/>
-    </joint>
-  </xacro:macro>
-  <xacro:drone id="1"/>
-  <xacro:drone id="2"/>
-  <xacro:drone id="3"/>
 </robot>

Commit message: wip: tf frames of multiple drones from config showing, but the cad model isnt

File: src/drone_viz/urdf/drone_arena.xacro (robot description, xacro)
@@ -3,5 +3,5 @@
   <link name="arena">
     <visual>
-      <origin xyz="0 0 0" rpy="0 0 0"/>
+      <origin xyz="0 0 1.3716" rpy="0 0 0"/>
       <geometry>
         <box size="6.7056 5.4864 2.7432"/>
@@ -12,5 +12,5 @@
     </visual>
   </link>
-  <link name="base_link">
+  <!-- <link name="base_link">
     <visual>
       <geometry>
@@ -23,4 +23,22 @@
     <child link="base_link"/>
     <origin xyz="0 0 -2.7432" rpy="0 0 0"/>
-  </joint>
+  </joint> -->
+  <xacro:macro name="drone_instance" params="name mesh">
+    <link name="${name}_base_link">
+      <visual>
+        <geometry>
+          <mesh filename="package://drone_viz/meshes/${mesh}" scale="0.1 0.1 0.1"/>
+        </geometry>
+        <material name="gray">
+          <color rgba="1 0 0"/>
+        </material>
+      </visual>
+    </link>
+    <joint name="${name}_joint" type="fixed">
+      <parent link="arena"/>
+      <child link="${name}_base_link"/>
+      <origin xyz="0 0 0" rpy="0 0 0"/>
+    </joint>
+  </xacro:macro>
+  <!-- <xacro:include filename="$(find drone_viz)/urdf/drone_params.xacro"/> -->
 </robot>
